File: geo_lpc1114.kicad_sch (KiCad schematic)
At the start: 143 parts, among them J1 CN_SWD, J10 Screw_Terminal_01x02, J11 Screw_Terminal_01x02, J12 Screw_Terminal_01x02, J13 Screw_Terminal_01x02, J14 Screw_Terminal_01x02, J15 Screw_Terminal_01x02, J16 Screw_Terminal_01x02, J17 Screw_Terminal_01x02, J18 USB_B, J19 MJ-179PH, J2 Screw_Terminal_01x02, J3 Screw_Terminal_01x02, J4 Screw_Terminal_01x02, J5 Screw_Terminal_01x02, J6 Screw_Terminal_01x02, J7 Screw_Terminal_01x02, J8 Screw_Terminal_01x02, J9 Screw_Terminal_01x02, Q1 S8550, Q2 S8550, Q3 S8550, Q4 S8550, Q5 S8550, Q6 S8550, Q7 S8550, Q8 S8550, SW1 SW, U1 LPC1114FN28-102, U10 LPC1114FDH28-102, U11 CH340N, U12 LM2940T-3.3, U2 HX711, U3 HX711, U4 HX711, U5 HX711, U6 HX711, U7 HX711, U8 HX711, U9 HX711, Y1 ZZT 12.0MT-22P

Commit message: fubriaction version 2024/09 1st week
Parts:
- removed D8: LED, LED_THT:LED_D3.0mm, symbol Device:LED
- removed J2, J3, J4, J5: Screw_Terminal_01x02, TerminalBlock:TerminalBlock_Xinya_XY308-2.54-2P_1x02_P2.54mm_Horizontal, symbol Connector:Screw_Terminal_01x02
- removed Q1, Q2: S8550, Package_TO_SOT_THT:TO-92_HandSolder, symbol Transistor_BJT:S8550
- removed R10, R6, R9: 20k, Resistor_THT:R_Axial_DIN0204_L3.6mm_D1.6mm_P7.62mm_Horizontal, symbol Device:R
- removed R11, R12: 100, Resistor_THT:R_Axial_DIN0204_L3.6mm_D1.6mm_P7.62mm_Horizontal, symbol Device:R
- removed R13, R14, R7, R8: 20, Resistor_THT:R_Axial_DIN0204_L3.6mm_D1.6mm_P7.62mm_Horizontal, symbol Device:R
- removed R51: 10k, Resistor_THT:R_Axial_DIN0204_L3.6mm_D1.6mm_P7.62mm_Horizontal, symbol Device:R
- removed U2, U3: HX711, Package_SO:SOIC-16_3.9x9.9mm_P1.27mm, symbol Analog_ADC:HX711
- removed Y1: ZZT 12.0MT-22P, Crystal:Crystal_HC52-U-3Pin_Vertical, symbol Device:Crystal_GND2
- added J2: AQM1602Y-NLW-FBW, Connector_PinHeader_2.54mm:PinHeader_1x09_P2.54mm_Vertical, symbol Connector_Generic:Conn_01x09
- added J3: GPIO_Header, Connector_PinHeader_2.54mm:PinHeader_1x04_P2.54mm_Vertical, symbol Connector:Conn_01x04_Pin
- added J4: I2C_Header, Connector_PinHeader_2.54mm:PinHeader_1x04_P2.54mm_Vertical, symbol Connector:Conn_01x04_Pin
- added J5: UART_Header, Connector_PinHeader_2.54mm:PinHeader_1x04_P2.54mm_Vertical, symbol Connector:Conn_01x04_Pin
- added SW2: SW, Button_Switch_THT:SW_TH_Tactile_Omron_B3F-100x, symbol Switch:SW_Omron_B3FS
- added Y1: 12MHz, Crystal:Crystal_HC49-U_Vertical, symbol Device:Crystal
- C10, C11: value 0.1μF 50V X7R -> 22pF; footprint Capacitor_THT:C_Disc_D3.8mm_W2.6mm_P2.50mm -> Capacitor_THT:C_Disc_D4.3mm_W1.9mm_P5.00mm
- C4, C5: value 10μF 16V X7R -> 0.1μF 50V X7R; footprint Capacitor_THT:C_Disc_D5.1mm_W3.2mm_P5.00mm -> Capacitor_THT:C_Disc_D3.8mm_W2.6mm_P2.50mm
- C7: value 0.1μF 50V X7R -> 1μF 50V X7R; footprint Capacitor_THT:C_Disc_D3.8mm_W2.6mm_P2.50mm -> Capacitor_THT:C_Disc_D4.3mm_W1.9mm_P5.00mm
- C8, C9: value 10μF 16V X7R -> 1μF 50V X7R; footprint Capacitor_THT:C_Disc_D5.1mm_W3.2mm_P5.00mm -> Capacitor_THT:C_Disc_D4.3mm_W1.9mm_P5.00mm
- R1: value 4.7k -> 10k
- R3, R4: value 100 -> 10k
- R5: value 20k -> 10k
Connections:
- net HX711_CLK_6 is gone; now on net HX711_CLK_4: R38.1, U1.17 (PIO1_8), U10.17 (PIO1_8)
- net HX711_CLK_7 is gone; now on net HX711_CLK_5: R50.1, U1.14 (PIO1_5), U10.14 (PIO1_5)
- net HX711_DAT_6 is gone; now on net HX711_DAT_4: R37.2, U1.18 (PIO1_9), U10.18 (PIO1_9)
- net HX711_DAT_7 is gone; now on net HX711_DAT_5: R49.2, U1.13 (PIO1_4), U10.13 (PIO1_4)
- net +3V3: now also C4.1, C5.1, C6.1, C8.2, C9.1, R3.1, R4.1, R5.1, J2.5 (Pin_5), J3.4 (Pin_4), J4.4 (Pin_4), J5.4 (Pin_4); no longer C11.2, C7.2
- net GND: now also C11.2, C4.2, C9.2, J2.4 (Pin_4), J3.1 (Pin_1), J4.1 (Pin_1), J5.1 (Pin_1), SW2.1; no longer C11.1, C7.1, C8.2
- net HX711_CLK_0: now also R20.1
- net HX711_CLK_1: now also R26.1, U1.4 (PIO0_11), U10.4 (PIO0_11); no longer U1.5 (PIO0_5/SDA), U10.5 (PIO0_5/SDA)
- net HX711_CLK_2: now also R36.1, U1.9 (PIO1_0), U10.9 (PIO1_0); no longer R20.1, U1.27 (PIO0_4/SCK), U10.27 (PIO0_4/SCK)
- net HX711_CLK_3: now also R48.1, U1.11 (PIO1_2), U10.11 (PIO1_2); no longer R26.1, U1.25 (PIO0_2), U10.25 (PIO0_2)
- net HX711_CLK_4: no longer R36.1, U1.9 (PIO1_0), U10.9 (PIO1_0)
- net HX711_CLK_5: no longer R48.1, U1.11 (PIO1_2), U10.11 (PIO1_2)
- net HX711_DAT_0: now also R19.2
- net HX711_DAT_1: now also R25.2, U1.25 (PIO0_2), U10.25 (PIO0_2); no longer U1.4 (PIO0_11), U10.4 (PIO0_11)
- net HX711_DAT_2: now also R35.2, U1.6 (PIO0_6), U10.6 (PIO0_6); no longer R19.2, U1.28 (PIO0_7), U10.28 (PIO0_7)
- net HX711_DAT_3: now also R47.2, U1.10 (PIO1_1), U10.10 (PIO1_1); no longer R25.2, U1.26 (PIO0_3), U10.26 (PIO0_3)
- net HX711_DAT_4: no longer R35.2, U1.6 (PIO0_6), U10.6 (PIO0_6)
- net HX711_DAT_5: no longer R47.2, U1.10 (PIO1_1), U10.10 (PIO1_1)
- net UART_RX: now also J5.2 (Pin_2)
- net UART_TX: now also J5.3 (Pin_3)
- net XTAL_IN: now also C10.1, Y1.2
- net XTAL_OUT: now also C11.1, Y1.1
- net I2C_SDA: now reaches R3.2
- net I2C_SDA: now also U1.5 (PIO0_5/SDA), U10.5 (PIO0_5/SDA), J2.3 (Pin_3), J4.2 (Pin_2); no longer C4.1
- net I2C_SCL: now reaches R4.2
- net I2C_SCL: now also U1.27 (PIO0_4/SCK), U10.27 (PIO0_4/SCK), J2.2 (Pin_2), J4.3 (Pin_3); no longer C4.2
- net at R5.2: now also J2.1 (Pin_1); no longer C5.1
- net at C8.1: now also J2.6 (Pin_6)
- net LED renamed ISP/LED
- net ISP/LED: now also SW2.2
- new net: C7.2, J2.7 (Pin_7)
- new net: C7.1, J2.8 (Pin_8)
- new net PIO0_3: J3.2 (Pin_2), U1.26 (PIO0_3), U10.26 (PIO0_3)
- new net PIO0_7: J3.3 (Pin_3), U1.28 (PIO0_7), U10.28 (PIO0_7)
- no-connect marks 9 -> 8
Other:
- moved on the sheet: C1, C12, C13, C14, C15, C16, C17, C18, C19, C2, C20, C21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
